File: surface-mount/pico-dirty-blaster-sm.kicad_sch (KiCad schematic)
At the start: 4 parts, among them J1 Conn_01x06, J2 Conn_02x05_Counter_Clockwise, J3 Conn_02x05_Counter_Clockwise

Commit message: connected vcc on SM, 0402 R on LS
Connections:
- net J_VCC: now reaches J3.4 (Pin_4)
- net J_VCC: now also J2.1 (Pin_1)
Changed lines of the file:
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@@
+    (stroke (width 0) (type default))
+  )
+  (wire (pts (xy 127 167.64) (xy 132.08 167.64))
     (stroke (width 0) (type default))
   )
@@
   )
   (wire (pts (xy 50.8 152.4) (xy 86.36 152.4))
+    (stroke (width 0) (type default))
+  )
+  (wire (pts (xy 132.08 167.64) (xy 132.08 160.02))
     (stroke (width 0) (type default))
   )
@@
     (stroke (width 0) (type default))
   )
+  (wire (pts (xy 55.88 160.02) (xy 55.88 165.1))
+    (stroke (width 0) (type default))
+  )
   (wire (pts (xy 53.34 147.32) (xy 53.34 167.64))
     (stroke (width 0) (type default))
   )
   (wire (pts (xy 101.6 175.26) (xy 101.6 152.4))
+    (stroke (width 0) (type default))
+  )
+  (wire (pts (xy 55.88 165.1) (xy 63.5 165.1))
     (stroke (width 0) (type default))
   )
@@
   )
   (wire (pts (xy 50.8 147.32) (xy 53.34 147.32))
+    (stroke (width 0) (type default))
+  )
+  (wire (pts (xy 132.08 160.02) (xy 55.88 160.02))
     (stroke (width 0) (type default))
   )
@@
     (effects (font (size 1.27 1.27)) (justify left bottom))
   )
+  (label "J_VCC" (at 55.88 160.02 0) (fields_autoplaced)
+    (effects (font (size 1.27 1.27)) (justify left bottom))
+  )
